File: Eagle PCB/PB.sch (EAGLE design)
At the start: 25 parts, among them IC1 74HC595D, IC2 74HC595D, IC3 L78LXXCU/BU, J1 61300511121, J2 61300211121, J3 61300211121, J4 61300511121, J5 61300211121, J6 61300511121, J7 61300211121

Commit message: Final PCB schematic and board added.
Parts:
- removed J3, J5: 61300211121, Headers:61300211121
- added JP1, JP2, JP3, JP4, JP5, JP6: (no value), pinhead:PINHD-1X1
Connections:
- net N$11 renamed SA
- removed net GND: IC3.GND1
- removed net N$1: IC1A.RCK, J2.2
- removed net N$12: IC2A.SER, J3.1
- removed net N$25: IC2A.RCK, J3.2
- new net OE: IC1A.G, IC2A.G, JP1.1, JP4.1
- new net RCK: IC1A.RCK, IC2A.RCK, JP2.1, JP5.1
- new net SB: IC2A.SER, J2.2
- net 0: now also IC3.GND1; no longer IC1A.G, IC2A.G, J5.2
- net CLK: now also JP3.1, JP6.1
- net VCC: no longer J5.1
Other:
- moved on the sheet: J2, J7

Commit message: PCB updated with common serial input.
Parts:
- removed C1, C4, C7: 10uF, SparkFun-Capacitors:10UF-0603-6.3V-20%
- removed J2: 61300211121, Headers:61300211121
- added C10, C11, C12: 10uF, SparkFun-Capacitors:10UF-0805-10V-10%
- added JP7, JP8: (no value), pinhead:PINHD-1X1
Connections:
- new net N$1: IC2A.QH*, JP8.1
- net 0: now also C10.2, C11.2, C12.2; no longer C1.2, C4.2, C7.2
- net SA: now also JP7.1; no longer J2.1
- net SB: now also IC1A.QH*; no longer J2.2
- net VDD: now also C10.1, C11.1, C12.1; no longer C1.1, C4.1, C7.1
